Commit message: Completed motors on creatures

File: test.urdf (robot description, URDF)
Before this commit: robot creature, 12 links, 11 joints
Links:
- removed link 15
- removed link 24
- removed link 26
- removed link 27
- removed link 28
- removed link 310
- removed link 311
- removed link 39
- added link 34, mass 0.36344713145753615; collision cylinder length=0.5310067609003892 radius=0.46676218165266425; visual cylinder length=0.5310067609003892 radius=0.46676218165266425
- link 0: mass 2.039892591272529 -> 0.42710706426258266; geometry collision cylinder length=0.5182380051505815 radius=0.5121873068740359; visual cylinder length=0.5182380051505815 radius=0.5121873068740359
- link 11: mass 1.7617049951617743 -> 5.8683389505843215e-05; geometry collision cylinder length=0.41000644112793194 radius=0.0067497442738964075; visual cylinder length=0.41000644112793194 radius=0.0067497442738964075
- link 22: mass 0.3497181964780981 -> 0.0021617846191605197; geometry collision cylinder length=0.28414969748898256 radius=0.049210488470198266; visual cylinder length=0.28414969748898256 radius=0.049210488470198266
- link 23: mass 0.3497181964780981 -> 0.0021617846191605197; geometry collision cylinder length=0.28414969748898256 radius=0.049210488470198266; visual cylinder length=0.28414969748898256 radius=0.049210488470198266
Joints:
- removed joint 15_to_0
- removed joint 22_to_11
- removed joint 23_to_11
- removed joint 24_to_11
- removed joint 26_to_15
- removed joint 27_to_15
- removed joint 28_to_15
- removed joint 310_to_0
- removed joint 311_to_0
- removed joint 39_to_0
- added joint 22_to_0: type revolute, parent 0, child 22, origin xyz=0.8713441982706265 0.549129525004211 0.16081124121088508 rpy=17.07247146151459 1.8213841877370438 3.5211809265038676, axis 0 1 0, limit lower=0 upper=1 effort=1 velocity=1
- added joint 23_to_0: type revolute, parent 0, child 23, origin xyz=0.8713441982706265 0.549129525004211 0.16081124121088508 rpy=22.763295282019453 1.8213841877370438 3.5211809265038676, axis 0 1 0, limit lower=0 upper=1 effort=1 velocity=1
- added joint 34_to_0: type revolute, parent 0, child 34, origin xyz=0.2056852189627143 0.3760083842404496 0.571554866267603 rpy=18.584277935540136 2.091328759636623 1.0416123087715878, axis 1 0 0, limit lower=0 upper=1 effort=1 velocity=1
- joint 11_to_0: axis 0 1 0 -> 0 0 1; origin xyz=0.49432203096411664 0.8707948391526354 0.869944583055941 rpy=6.033323382883783 1.8522425330580654 1.0537502037244184 -> xyz=0.5793881670103216 0.8364341932181882 0.23611581791492153 rpy=5.719137843066718 3.496186034462074 3.920960893675664

Commit message: Confirmed motors work on creature

File: test.urdf (robot description, URDF)
Before this commit: robot creature, 5 links, 4 joints
Links:
- removed link 34
- added link 113, mass 0.17172568823209855; collision cylinder length=0.6738426916824442 radius=0.28481537852536964; visual cylinder length=0.6738426916824442 radius=0.28481537852536964
- added link 15, mass 0.17172568823209855; collision cylinder length=0.6738426916824442 radius=0.28481537852536964; visual cylinder length=0.6738426916824442 radius=0.28481537852536964
- added link 19, mass 0.17172568823209855; collision cylinder length=0.6738426916824442 radius=0.28481537852536964; visual cylinder length=0.6738426916824442 radius=0.28481537852536964
- added link 210, mass 0.2885428417544324; collision cylinder length=0.286686317623689 radius=0.5660134259152717; visual cylinder length=0.286686317623689 radius=0.5660134259152717
- added link 211, mass 0.2885428417544324; collision cylinder length=0.286686317623689 radius=0.5660134259152717; visual cylinder length=0.286686317623689 radius=0.5660134259152717
- added link 212, mass 0.2885428417544324; collision cylinder length=0.286686317623689 radius=0.5660134259152717; visual cylinder length=0.286686317623689 radius=0.5660134259152717
- added link 214, mass 0.2885428417544324; collision cylinder length=0.286686317623689 radius=0.5660134259152717; visual cylinder length=0.286686317623689 radius=0.5660134259152717
- added link 215, mass 0.2885428417544324; collision cylinder length=0.286686317623689 radius=0.5660134259152717; visual cylinder length=0.286686317623689 radius=0.5660134259152717
- added link 216, mass 0.2885428417544324; collision cylinder length=0.286686317623689 radius=0.5660134259152717; visual cylinder length=0.286686317623689 radius=0.5660134259152717
- added link 24, mass 0.2885428417544324; collision cylinder length=0.286686317623689 radius=0.5660134259152717; visual cylinder length=0.286686317623689 radius=0.5660134259152717
- added link 26, mass 0.2885428417544324; collision cylinder length=0.286686317623689 radius=0.5660134259152717; visual cylinder length=0.286686317623689 radius=0.5660134259152717
- added link 27, mass 0.2885428417544324; collision cylinder length=0.286686317623689 radius=0.5660134259152717; visual cylinder length=0.286686317623689 radius=0.5660134259152717
- added link 28, mass 0.2885428417544324; collision cylinder length=0.286686317623689 radius=0.5660134259152717; visual cylinder length=0.286686317623689 radius=0.5660134259152717
- added link 317, mass 1.6693147679543876; collision cylinder length=0.5563614018216806 radius=0.9772725156201775; visual cylinder length=0.5563614018216806 radius=0.9772725156201775
- added link 318, mass 1.6693147679543876; collision cylinder length=0.5563614018216806 radius=0.9772725156201775; visual cylinder length=0.5563614018216806 radius=0.9772725156201775
- added link 319, mass 1.6693147679543876; collision cylinder length=0.5563614018216806 radius=0.9772725156201775; visual cylinder length=0.5563614018216806 radius=0.9772725156201775
- added link 320, mass 1.6693147679543876; collision cylinder length=0.5563614018216806 radius=0.9772725156201775; visual cylinder length=0.5563614018216806 radius=0.9772725156201775
- added link 421, mass 0.4131595611038684; collision cylinder length=0.2406959102839108 radius=0.7391789857995966; visual cylinder length=0.2406959102839108 radius=0.7391789857995966
- added link 422, mass 0.4131595611038684; collision cylinder length=0.2406959102839108 radius=0.7391789857995966; visual cylinder length=0.2406959102839108 radius=0.7391789857995966
- added link 423, mass 0.4131595611038684; collision cylinder length=0.2406959102839108 radius=0.7391789857995966; visual cylinder length=0.2406959102839108 radius=0.7391789857995966
- link 0: mass 0.42710706426258266 -> 0.024957978858026506; geometry collision cylinder length=0.8147594184432141 radius=0.09874499113039481; visual cylinder length=0.8147594184432141 radius=0.09874499113039481
- link 11: mass 5.8683389505843215e-05 -> 0.17172568823209855; geometry collision cylinder length=0.6738426916824442 radius=0.28481537852536964; visual cylinder length=0.6738426916824442 radius=0.28481537852536964
- link 22: mass 0.0021617846191605197 -> 0.2885428417544324; geometry collision cylinder length=0.286686317623689 radius=0.5660134259152717; visual cylinder length=0.286686317623689 radius=0.5660134259152717
- link 23: mass 0.0021617846191605197 -> 0.2885428417544324; geometry collision cylinder length=0.286686317623689 radius=0.5660134259152717; visual cylinder length=0.286686317623689 radius=0.5660134259152717
Joints:
- removed joint 22_to_0
- removed joint 23_to_0
- removed joint 34_to_0
- added joint 113_to_0: type revolute, parent 0, child 113, origin xyz=0.8513480815330349 0.3054509135256316 0.9762482853559791 rpy=1.25666935978321 4.198655501048746 5.3880503306581975, axis 1 0 0, limit lower=0 upper=1 effort=1 velocity=1
- added joint 15_to_0: type revolute, parent 0, child 15, origin xyz=0.8513480815330349 0.3054509135256316 0.9762482853559791 rpy=0.7540016158699259 4.198655501048746 5.3880503306581975, axis 1 0 0, limit lower=0 upper=1 effort=1 velocity=1
- added joint 19_to_0: type revolute, parent 0, child 19, origin xyz=0.8513480815330349 0.3054509135256316 0.9762482853559791 rpy=1.005335487826568 4.198655501048746 5.3880503306581975, axis 1 0 0, limit lower=0 upper=1 effort=1 velocity=1
- added joint 210_to_19: type fixed, parent 19, child 210, origin xyz=0.6046231336092414 0.48543060007811456 0.4798691802417 rpy=11.127429647094939 4.8014932081620065 2.4799414744329016, axis 1 0 0, limit lower=0 upper=1 effort=1 velocity=1
- added joint 211_to_19: type fixed, parent 19, child 211, origin xyz=0.6046231336092414 0.48543060007811456 0.4798691802417 rpy=16.691144470642406 4.8014932081620065 2.4799414744329016, axis 1 0 0, limit lower=0 upper=1 effort=1 velocity=1
- added joint 212_to_19: type fixed, parent 19, child 212, origin xyz=0.6046231336092414 0.48543060007811456 0.4798691802417 rpy=22.254859294189878 4.8014932081620065 2.4799414744329016, axis 1 0 0, limit lower=0 upper=1 effort=1 velocity=1
- added joint 214_to_113: type fixed, parent 113, child 214, origin xyz=0.6046231336092414 0.48543060007811456 0.4798691802417 rpy=11.127429647094939 4.8014932081620065 2.4799414744329016, axis 1 0 0, limit lower=0 upper=1 effort=1 velocity=1
- added joint 215_to_113: type fixed, parent 113, child 215, origin xyz=0.6046231336092414 0.48543060007811456 0.4798691802417 rpy=16.691144470642406 4.8014932081620065 2.4799414744329016, axis 1 0 0, limit lower=0 upper=1 effort=1 velocity=1
- added joint 216_to_113: type fixed, parent 113, child 216, origin xyz=0.6046231336092414 0.48543060007811456 0.4798691802417 rpy=22.254859294189878 4.8014932081620065 2.4799414744329016, axis 1 0 0, limit lower=0 upper=1 effort=1 velocity=1
- added joint 22_to_11: type fixed, parent 11, child 22, origin xyz=0.6046231336092414 0.48543060007811456 0.4798691802417 rpy=11.127429647094939 4.8014932081620065 2.4799414744329016, axis 1 0 0, limit lower=0 upper=1 effort=1 velocity=1
- added joint 23_to_11: type fixed, parent 11, child 23, origin xyz=0.6046231336092414 0.48543060007811456 0.4798691802417 rpy=16.691144470642406 4.8014932081620065 2.4799414744329016, axis 1 0 0, limit lower=0 upper=1 effort=1 velocity=1
- added joint 24_to_11: type fixed, parent 11, child 24, origin xyz=0.6046231336092414 0.48543060007811456 0.4798691802417 rpy=22.254859294189878 4.8014932081620065 2.4799414744329016, axis 1 0 0, limit lower=0 upper=1 effort=1 velocity=1
- added joint 26_to_15: type fixed, parent 15, child 26, origin xyz=0.6046231336092414 0.48543060007811456 0.4798691802417 rpy=11.127429647094939 4.8014932081620065 2.4799414744329016, axis 1 0 0, limit lower=0 upper=1 effort=1 velocity=1
- added joint 27_to_15: type fixed, parent 15, child 27, origin xyz=0.6046231336092414 0.48543060007811456 0.4798691802417 rpy=16.691144470642406 4.8014932081620065 2.4799414744329016, axis 1 0 0, limit lower=0 upper=1 effort=1 velocity=1
- added joint 28_to_15: type fixed, parent 15, child 28, origin xyz=0.6046231336092414 0.48543060007811456 0.4798691802417 rpy=22.254859294189878 4.8014932081620065 2.4799414744329016, axis 1 0 0, limit lower=0 upper=1 effort=1 velocity=1
- added joint 317_to_0: type fixed, parent 0, child 317, origin xyz=0.6002440498471823 0.17619078604030458 0.9476273352071014 rpy=23.980402148333628 1.7778522685852391 1.8208055921150152, axis 1 0 0, limit lower=0 upper=1 effort=1 velocity=1
- added joint 318_to_0: type fixed, parent 0, child 318, origin xyz=0.6002440498471823 0.17619078604030458 0.9476273352071014 rpy=27.977135839722564 1.7778522685852391 1.8208055921150152, axis 1 0 0, limit lower=0 upper=1 effort=1 velocity=1
- added joint 319_to_0: type fixed, parent 0, child 319, origin xyz=0.6002440498471823 0.17619078604030458 0.9476273352071014 rpy=31.973869531111504 1.7778522685852391 1.8208055921150152, axis 1 0 0, limit lower=0 upper=1 effort=1 velocity=1
- added joint 320_to_0: type fixed, parent 0, child 320, origin xyz=0.6002440498471823 0.17619078604030458 0.9476273352071014 rpy=35.97060322250044 1.7778522685852391 1.8208055921150152, axis 1 0 0, limit lower=0 upper=1 effort=1 velocity=1
- added joint 421_to_0: type fixed, parent 0, child 421, origin xyz=0.7177804657798312 0.711349240910306 0.03420204741864841 rpy=59.929082591721176 5.6324997439783 0.3503281877869593, axis 0 1 0, limit lower=0 upper=1 effort=1 velocity=1
- added joint 422_to_0: type fixed, parent 0, child 422, origin xyz=0.7177804657798312 0.711349240910306 0.03420204741864841 rpy=65.9219908508933 5.6324997439783 0.3503281877869593, axis 0 1 0, limit lower=0 upper=1 effort=1 velocity=1
- added joint 423_to_0: type fixed, parent 0, child 423, origin xyz=0.7177804657798312 0.711349240910306 0.03420204741864841 rpy=71.9148991100654 5.6324997439783 0.3503281877869593, axis 0 1 0, limit lower=0 upper=1 effort=1 velocity=1
- joint 11_to_0: axis 0 0 1 -> 1 0 0; origin xyz=0.5793881670103216 0.8364341932181882 0.23611581791492153 rpy=5.719137843066718 3.496186034462074 3.920960893675664 -> xyz=0.8513480815330349 0.3054509135256316 0.9762482853559791 rpy=0.502667743913284 4.198655501048746 5.3880503306581975
