Commit message: Implemented fitness function

File: temp.urdf (robot description, URDF)
Before this commit: robot creature, 6 links, 5 joints
Links:
- removed link 22
- removed link 23
- removed link 24
- added link 12, mass 0.5671763018272226; collision cylinder length=0.3569941865959124 radius=0.7111374169677014; visual cylinder length=0.3569941865959124 radius=0.7111374169677014
- added link 13, mass 0.5671763018272226; collision cylinder length=0.3569941865959124 radius=0.7111374169677014; visual cylinder length=0.3569941865959124 radius=0.7111374169677014
- added link 14, mass 0.5671763018272226; collision cylinder length=0.3569941865959124 radius=0.7111374169677014; visual cylinder length=0.3569941865959124 radius=0.7111374169677014
- added link 26, mass 1.3466131619055708; collision cylinder length=0.9755838030079949 radius=0.6628483819001386; visual cylinder length=0.9755838030079949 radius=0.6628483819001386
- link 0: mass 1.8009749775523782 -> 0.5895007856285224; geometry collision cylinder length=0.6632294759032492 radius=0.53190656195671; visual cylinder length=0.6632294759032492 radius=0.53190656195671
- link 11: mass 0.31578881875754206 -> 0.5671763018272226; geometry collision cylinder length=0.3569941865959124 radius=0.7111374169677014; visual cylinder length=0.3569941865959124 radius=0.7111374169677014
- link 25: mass 0.33723904045279574 -> 1.3466131619055708; geometry collision cylinder length=0.9755838030079949 radius=0.6628483819001386; visual cylinder length=0.9755838030079949 radius=0.6628483819001386
Joints:
- removed joint 22_to_11
- removed joint 23_to_11
- removed joint 24_to_11
- removed joint 25_to_11
- added joint 12_to_0: type fixed, parent 0, child 12, origin xyz=0.6488864803738003 0.894438255318445 0.39327005332560083 rpy=2.4183914009207417 3.675324512797596 3.8865406484329683, axis 0 1 0, limit lower=0 upper=1 effort=1 velocity=1
- added joint 13_to_0: type fixed, parent 0, child 13, origin xyz=0.6488864803738003 0.894438255318445 0.39327005332560083 rpy=3.224521867894322 3.675324512797596 3.8865406484329683, axis 0 1 0, limit lower=0 upper=1 effort=1 velocity=1
- added joint 14_to_0: type fixed, parent 0, child 14, origin xyz=0.6488864803738003 0.894438255318445 0.39327005332560083 rpy=4.030652334867902 3.675324512797596 3.8865406484329683, axis 0 1 0, limit lower=0 upper=1 effort=1 velocity=1
- added joint 25_to_0: type fixed, parent 0, child 25, origin xyz=0.5650924585737654 0.1065219207558733 0.6393257114651621 rpy=9.914206140468252 2.132995404275924 3.7944542197612385, axis 0 1 0, limit lower=0 upper=1 effort=1 velocity=1
- added joint 26_to_0: type fixed, parent 0, child 26, origin xyz=0.5650924585737654 0.1065219207558733 0.6393257114651621 rpy=11.566573830546295 2.132995404275924 3.7944542197612385, axis 0 1 0, limit lower=0 upper=1 effort=1 velocity=1
- joint 11_to_0: origin xyz=0.6958416647432165 0.004804272738273441 0.9201720907058762 rpy=1.2577299277350977 5.481256184935472 0.804077008332888 -> xyz=0.6488864803738003 0.894438255318445 0.39327005332560083 rpy=1.612260933947161 3.675324512797596 3.8865406484329683; type revolute -> fixed
