Commit message: Added offline simulation

File: temp0.urdf (robot description, URDF)
Before this commit: robot creature, 3 links, 2 joints
Links:
- removed link 22
- added link 12, mass 0.17343461569980534; collision cylinder length=0.2846492868542808 radius=0.44039046235374935; visual cylinder length=0.2846492868542808 radius=0.44039046235374935
- added link 13, mass 0.17343461569980534; collision cylinder length=0.2846492868542808 radius=0.44039046235374935; visual cylinder length=0.2846492868542808 radius=0.44039046235374935
- added link 14, mass 0.17343461569980534; collision cylinder length=0.2846492868542808 radius=0.44039046235374935; visual cylinder length=0.2846492868542808 radius=0.44039046235374935
- added link 25, mass 1.224772456223729; collision cylinder length=0.479149652014801 radius=0.9020221052056012; visual cylinder length=0.479149652014801 radius=0.9020221052056012
- link 0: mass 1.0302391330766618 -> 0.008372948203478787; geometry collision cylinder length=0.16909351415917828 radius=0.12554539603197934; visual cylinder length=0.16909351415917828 radius=0.12554539603197934
- link 11: mass 0.5822338920158273 -> 0.17343461569980534; geometry collision cylinder length=0.2846492868542808 radius=0.44039046235374935; visual cylinder length=0.2846492868542808 radius=0.44039046235374935
Joints:
- removed joint 22_to_11
- added joint 12_to_0: type revolute, parent 0, child 12, origin xyz=0.7997268607936372 0.5388188938303738 0.6976420407981926 rpy=17.076687450720407 0.816208611836453 6.215073736786412, axis 1 0 0, limit lower=0 upper=1 effort=1 velocity=1
- added joint 13_to_0: type revolute, parent 0, child 13, origin xyz=0.7997268607936372 0.5388188938303738 0.6976420407981926 rpy=22.768916600960544 0.816208611836453 6.215073736786412, axis 1 0 0, limit lower=0 upper=1 effort=1 velocity=1
- added joint 14_to_0: type revolute, parent 0, child 14, origin xyz=0.7997268607936372 0.5388188938303738 0.6976420407981926 rpy=28.461145751200682 0.816208611836453 6.215073736786412, axis 1 0 0, limit lower=0 upper=1 effort=1 velocity=1
- added joint 25_to_0: type fixed, parent 0, child 25, origin xyz=0.1664432173552205 0.6254807393135818 0.5140311348546337 rpy=10.396541789598285 1.3211997606909127 1.566092005974654, axis 1 0 0, limit lower=0 upper=1 effort=1 velocity=1
- joint 11_to_0: axis 0 1 0 -> 1 0 0; origin xyz=0.17653748874779107 0.3440860502999834 0.7451131631765382 rpy=9.867897497662396 5.159269839627949 0.7362513629478991 -> xyz=0.7997268607936372 0.5388188938303738 0.6976420407981926 rpy=11.384458300480272 0.816208611836453 6.215073736786412; type fixed -> revolute
